File: hardware/Projet Wall E/projet/puissance.kicad_sch (KiCad schematic)
At the start: 0 parts

Commit message: feat(puissance): integration du schema de puissance termine
Parts:
- added C12: 0.01uF, Capacitor_SMD:C_01005_0402Metric, symbol Device:C_Small
- added C23: 2.2uF, Capacitor_SMD:C_01005_0402Metric, symbol Device:C_Small
- added C24: 10uF, Package_SO:SOIC-8_3.9x4.9mm_P1.27mm, symbol Device:C_Polarized_Small
- added J4, J5: Conn_01x06, Connector_JST:JST_VH_S6P-VH_1x06_P3.96mm_Horizontal, symbol Connector_Generic:Conn_01x06
- added R15, R16: 200m, symbol Device:R_Small
- added U5: DRV8833PWP, Package_SO:HTSSOP-16-1EP_4.4x5mm_P0.65mm_EP3.4x5mm_Mask2.46x2.31mm_ThermalVias, symbol Driver_Motor:DRV8833PWP
Connections:
- new net: R16.2, U5.6 (BISEN)
- new net: C23.2, U5.14 (VINT)
- new net: C12.2, U5.11 (VCP)
- new net: R15.2, U5.3 (AISEN)
- new net +3.3V: J4.5 (Pin_5), J5.5 (Pin_5)
- new net +5V: C12.1, C24.1, U5.12 (VM)
- new net AIN1: U5.16 (AIN1)
- new net AIN2: U5.15 (AIN2)
- new net AOUT1: J4.1 (Pin_1), U5.2 (AOUT1)
- new net AOUT2: J4.6 (Pin_6), U5.4 (AOUT2)
- new net BIN1: U5.9 (BIN1)
- new net BIN2: U5.10 (BIN2)
- new net BOUT1: J5.1 (Pin_1), U5.7 (BOUT1)
- new net BOUT2: J5.6 (Pin_6), U5.5 (BOUT2)
- new net ENCA_AOUT: J4.3 (Pin_3)
- new net ENCA_BOUT: J5.3 (Pin_3)
- new net ENCB_AOUT: J4.4 (Pin_4)
- new net ENCB_BOUT: J5.4 (Pin_4)
- new net GND: C23.1, C24.2, J4.2 (Pin_2), J5.2 (Pin_2), R15.1, R16.1, U5.13 (GND), U5.17 (GND)
- new net nFAULT: U5.8 (~{FAULT})
- new net nSleep: U5.1 (~{SLEEP})
Other:
- note added: "ENCODER"
- note added: "MOTOR DRIVER"

Commit message: feat(puissance): schema de puissance
Parts:
- removed C24: 10uF, Package_SO:SOIC-8_3.9x4.9mm_P1.27mm, symbol Device:C_Polarized_Small
- added C13: 10u, Capacitor_SMD:C_01005_0402Metric, symbol Device:C_Small
- added C14: 470u, Capacitor_SMD:C_01005_0402Metric, symbol Device:C_Small
- C12: value 0.01uF -> 10n
- R15, R16: footprint (none) -> Resistor_SMD:R_0201_0603Metric
Connections:
- net +3.3V: now also J4.2 (Pin_2), J5.2 (Pin_2); no longer J4.5 (Pin_5), J5.5 (Pin_5)
- net +5V: now also C13.1, C14.1
- net GND: now also J4.5 (Pin_5), J5.5 (Pin_5), C13.2, C14.2; no longer J4.2 (Pin_2), J5.2 (Pin_2)
- net nSleep renamed nSLEEP
