File: hardware/Projet Wall E/projet/mcu.kicad_sch (KiCad schematic)
At the start: 20 parts, among them J1 Conn_01x03, J2 Conn_ST_STDC14, U4 STM32G431RBTx, Y1 16MHz

Commit message: Petite modif MCU
Parts:
- U4: JLCPCB Parts (none) -> C431633
Changed lines of the file:
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@@
+			)
+		)
+		(property "JLCPCB Parts" "C431633"
+			(at 165.1 111.76 0)
+			(hide yes)
+			(show_name no)
+			(do_not_autoplace no)
+			(effects
+				(font
+					(size 1.27 1.27)
+				)
 			)
 		)

Commit message: Petite modif MCU
Parts:
- U4: JLCPCB Part# (none) -> C431633; JLCPCB Parts C431633 -> (none)
Changed lines of the file:
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@@
 			)
 		)
-		(property "JLCPCB Parts" "C431633"
+		(property "JLCPCB Part#" "C431633"
 			(at 165.1 111.76 0)
 			(hide yes)

Commit message: Annotation par feuille + références JLCPCB Part #
Parts:
- C301: renamed from C15; JLCPCB Part# C15195 -> C1525
- C302: renamed from C16; JLCPCB Part# C15195 -> C1525
- C303: renamed from C17; JLCPCB Part# C15195 -> C1525
- C304: renamed from C18; JLCPCB Part# C15195 -> C1525
- C305: renamed from C19; JLCPCB Part# C15195 -> C19666
- C306: renamed from C20; JLCPCB Part# C15195 -> C15195
- C307: renamed from C22; JLCPCB Part# C15195 -> C52923
- C308: renamed from C31; JLCPCB Part# C15195 -> C1525
- C309: renamed from C33; JLCPCB Part# C15195 -> C1525
- C310: renamed from C32; JLCPCB Part# C15195 -> C1545
- C311: renamed from C21; JLCPCB Part# C15195 -> C1545
- C312: renamed from C23; JLCPCB Part# C15195 -> C52923
- D301: renamed from D2; JLCPCB Part # C2286 -> (none); JLCPCB Part# (none) -> C2286
- D302: renamed from D1; JLCPCB Part # C2286 -> (none); JLCPCB Part# (none) -> C2286
- J302: renamed from J1; JLCPCB Part# (none) -> C49257
- R301: renamed from R3; JLCPCB Part # C11702 -> (none); JLCPCB Part# (none) -> C11702
- R302: renamed from R4; JLCPCB Part # C11702 -> (none); JLCPCB Part# (none) -> C11702
- Y301: renamed from Y1; JLCPCB Part # C13738 -> (none); JLCPCB Part# (none) -> C13738
- renumbered J2 to J301, U4 to U301

Commit message: Feuille racine : liaisons hiérarchiques + corrections ERC
Connections:
- net GAUGE_INT: now reaches U301.36 (PB14)
- net CHG_PG: now reaches U301.37 (PB15)
- net USB_DM: now reaches U301.45 (PA11)
- net USB_DP: now reaches U301.46 (PA12)
- net CHG_nCE: no longer names the net of U301.33 (PB11)
- no-connect marks 2 -> 19
Changed lines of the file:
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@@
+	)
+	(no_connect
+		(at 182.88 127)
+	)
+	(no_connect
+		(at 147.32 99.06)
+	)
+	(no_connect
+		(at 147.32 93.98)
+	)
+	(no_connect
+		(at 182.88 88.9)
+	)
+	(no_connect
+		(at 182.88 124.46)
+	)
+	(no_connect
+		(at 147.32 101.6)
+	)
+	(no_connect
+		(at 182.88 81.28)
+	)
+	(no_connect
+		(at 147.32 132.08)
+	)
+	(no_connect
+		(at 147.32 88.9)
+	)
+	(no_connect
+		(at 182.88 142.24)
+	)
+	(no_connect
+		(at 182.88 71.12)
+	)
+	(no_connect
+		(at 182.88 86.36)
+	)
+	(no_connect
+		(at 147.32 124.46)
+	)
+	(no_connect
+		(at 147.32 127)
 	)
 	(no_connect
@@
 	)
 	(no_connect
+		(at 147.32 129.54)
+	)
+	(no_connect
+		(at 147.32 96.52)
+	)
+	(no_connect
 		(at 44.45 120.65)
 	)
+	(no_connect
+		(at 182.88 73.66)
+	)
 	(wire
 		(pts
@@
 	(wire
 		(pts
+			(xy 185.42 152.4) (xy 182.88 152.4)
+		)
+		(stroke
+			(width 0)
+			(type default)
+		)
+	)
+	(wire
+		(pts
 			(xy 72.39 59.69) (xy 72.39 64.77)
 		)
@@
 	(wire
 		(pts
+			(xy 190.5 101.6) (xy 182.88 101.6)
+		)
+		(stroke
+			(width 0)
+			(type default)
+		)
+	)
+	(wire
+		(pts
 			(xy 72.39 64.77) (xy 57.15 64.77)
 		)
@@
 	(wire
 		(pts
+			(xy 190.5 99.06) (xy 182.88 99.06)
+		)
+		(stroke
+			(width 0)
+			(type default)
+		)
+	)
+	(wire
+		(pts
 			(xy 43.18 45.72) (xy 43.18 52.07)
 		)
@@
 	(wire
 		(pts
-			(xy 186.69 142.24) (xy 182.88 142.24)
-		)
-		(stroke
-			(width 0)
-			(type default)
-		)
-	)
-	(wire
-		(pts
 			(xy 57.15 45.72) (xy 43.18 45.72)
 		)
@@
 		(pts
 			(xy 100.33 45.72) (xy 88.9 45.72)
+		)
+		(stroke
+			(width 0)
+			(type default)
+		)
+	)
+	(wire
+		(pts
+			(xy 182.88 149.86) (xy 185.42 149.86)
 		)
 		(stroke
@@
 		)
 	)
+	(label "SERVO_PWM"
+		(at 187.96 129.54 0)
+		(effects
+			(font
+				(size 1.27 1.27)
+			)
+			(justify left bottom)
+		)
+	)
 	(label "SWDIO"
 		(at 186.69 104.14 0)
@@
 			)
 			(justify left bottom)
+		)
+	)
+	(label "SERVO_PWM"
+		(at 243.84 127 180)
+		(effects
+			(font
+				(size 1.27 1.27)
+			)
+			(justify right bottom)
 		)
 	)
@@
 		)
 	)
+	(hierarchical_label "CHG_PG"
+		(shape input)
+		(at 185.42 152.4 0)
+		(effects
+			(font
+				(size 1.27 1.27)
+			)
+			(justify left)
+		)
+	)
 	(hierarchical_label "SCL_CAPT"
 		(shape bidirectional)
@@
 		)
 	)
+	(hierarchical_label "USB_DM"
+		(shape bidirectional)
+		(at 190.5 99.06 0)
+		(effects
+			(font
+				(size 1.27 1.27)
+			)
+			(justify left)
+		)
+	)
 	(hierarchical_label "TOF_R_SHUT"
 		(shape output)
@@
 		)
 	)
-	(hierarchical_label "SERVO_PWM"
-		(shape output)
-		(at 187.96 129.54 0)
+	(hierarchical_label "GAUGE_INT"
+		(shape input)
+		(at 185.42 149.86 0)
 		(effects
 			(font
@@
 		)
 	)
-	(hierarchical_label "CHG_nCE"
-		(shape output)
-		(at 186.69 142.24 0)
-		(effects
-			(font
-				(size 1.27 1.27)
-			)
-			(justify left)
-		)
-	)
 	(hierarchical_label "ENCA_BOUT"
 		(shape input)
@@
 		)
 	)
-	(hierarchical_label "SERVO_PWM"
-		(shape output)
-		(at 243.84 127 180)
-		(effects
-			(font
-				(size 1.27 1.27)
-			)
-			(justify right)
-		)
-	)
 	(hierarchical_label "TOF_R_GPIO1"
 		(shape input)
@@
 		)
 	)
+	(hierarchical_label "USB_DP"
+		(shape bidirectional)
+		(at 190.5 101.6 0)
+		(effects
+			(font
+				(size 1.27 1.27)
+			)
+			(justify left)
+		)
+	)

Commit message: Modifs schématique
Connections:
- net VBUS renamed +5V_USB
Changed lines of the file:
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@@
+	)
+	(symbol
+		(lib_id "power:+5V")
+		(at 224.79 121.92 0)
+		(unit 1)
+		(body_style 1)
+		(exclude_from_sim no)
+		(in_bom yes)
+		(on_board yes)
+		(in_pos_files yes)
+		(dnp no)
+		(property "Reference" "#PWR0307"
+			(at 224.79 125.73 0)
+			(hide yes)
+			(show_name no)
+			(do_not_autoplace no)
+			(effects
+				(font
+					(size 1.27 1.27)
+				)
+			)
+		)
+		(property "Value" "+5V_USB"
+			(at 224.79 117.856 0)
+			(show_name no)
+			(do_not_autoplace no)
+			(effects
+				(font
+					(size 1.27 1.27)
+				)
+			)
+		)
+		(property "Footprint" ""
+			(at 224.79 121.92 0)
+			(hide yes)
+			(show_name no)
+			(do_not_autoplace no)
+			(effects
+				(font
+					(size 1.27 1.27)
+				)
+			)
+		)
+		(property "Datasheet" ""
+			(at 224.79 121.92 0)
+			(hide yes)
+			(show_name no)
+			(do_not_autoplace no)
+			(effects
+				(font
+					(size 1.27 1.27)
+				)
+			)
+		)
+		(property "Description" "Power symbol creates a global label with name \"+5V\""
+			(at 224.79 121.92 0)
+			(hide yes)
+			(show_name no)
+			(do_not_autoplace no)
+			(effects
+				(font
+					(size 1.27 1.27)
+				)
+			)
+		)
+		(pin "1"
+		)
+		(instances
+			(project "projet"
+				(path "/aad9219d-d686-4d68-8dbb-b3c2b0727159/8d7235a3-ed0d-4c0c-a716-b22c65fe70a8"
+					(reference "#PWR0307")
+					(unit 1)
+				)
+			)
+		)
 	)
 	(symbol
@@
 					(unit 1)
 				)
-			)
-		)
-	)
-	(symbol
-		(lib_id "power:+3.3V")
-		(at 224.79 121.92 0)
-		(unit 1)
-		(body_style 1)
-		(exclude_from_sim no)
-		(in_bom yes)
-		(on_board yes)
-		(in_pos_files yes)
-		(dnp no)
-		(fields_autoplaced yes)
-		(property "Reference" "#PWR0307"
-			(at 224.79 125.73 0)
-			(hide yes)
-			(show_name no)
-			(do_not_autoplace no)
-			(effects
-				(font
-					(size 1.27 1.27)
-				)
-			)
-		)
-		(property "Value" "VBUS"
-			(at 227.33 120.6499 0)
-			(show_name no)
-			(do_not_autoplace no)
-			(effects
-				(font
-					(size 1.27 1.27)
-				)
-				(justify left)
-			)
-		)
-		(property "Footprint" ""
-			(at 224.79 121.92 0)
-			(hide yes)
-			(show_name no)
-			(do_not_autoplace no)
-			(effects
-				(font
-					(size 1.27 1.27)
-				)
-			)
-		)
-		(property "Datasheet" ""
-			(at 224.79 121.92 0)
-			(hide yes)
-			(show_name no)
-			(do_not_autoplace no)
-			(effects
-				(font
-					(size 1.27 1.27)
-				)
-			)
-		)
-		(property "Description" "Power symbol creates a global label with name \"+3.3V\""
-			(at 224.79 121.92 0)
-			(hide yes)
-			(show_name no)
-			(do_not_autoplace no)
-			(effects
-				(font
-					(size 1.27 1.27)
-				)
-			)
-		)
-		(pin "1"
-		)
-		(instances
-			(project "projet"
-				(path "/aad9219d-d686-4d68-8dbb-b3c2b0727159/8d7235a3-ed0d-4c0c-a716-b22c65fe70a8"
-					(reference "#PWR0307")
-					(unit 1)
-				)
-			)
-			(project "mcu"
-				(path "/d1f6b90d-1ee5-4a93-8c97-f2b0d96541e8"
-					(reference "#PWR034")
-					(unit 1)
-				)

Commit message: WIP : MCU et config software (en cours)
Parts:
- added R303: 10k, Resistor_SMD:R_0402_1005Metric, symbol wall_e:R
Connections:
- net ENCA_AOUT: now also U301.20 (PA6); no longer U301.62 (PB9)
- net ENCA_BOUT: now also U301.12 (PA0); no longer U301.44 (PA10)
- net ENCB_AOUT: now also U301.21 (PA7); no longer U301.61 (PB8)
- net ENCB_BOUT: now also U301.13 (PA1); no longer U301.43 (PA9)
- net GND: now also R303.1
- net SCL_CAPT: now also U301.43 (PA9); no longer U301.22 (PC4)
- new net BOOT0: R303.2, U301.61 (PB8)
- no-connect marks 19 -> 17

Commit message: Schéma : 0 erreur ERC, pinout MCU finalisé + config .ioc
Parts:
- renumbered R303 to R301, R301 to R302, R302 to R303
Connections:
- net GAUGE_INT: now also U301.58 (PB5); no longer U301.36 (PB14)
- net TOF_R_SHUT renamed TOF_R_XSHUT
- new net NEOPIXEL: U301.36 (PB14)
Changed lines of the file:
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@@
 	)
 	(no_connect
-		(at 182.88 127)
-	)
-	(no_connect
 		(at 147.32 99.06)
 	)
@@
 	)
 	(no_connect
+		(at 182.88 137.16)
+	)
+	(no_connect
 		(at 182.88 124.46)
 	)
@@
 	(wire
 		(pts
+			(xy 186.69 127) (xy 182.88 127)
+		)
+		(stroke
+			(width 0)
+			(type default)
+		)
+	)
+	(wire
+		(pts
 			(xy 60.96 40.64) (xy 60.96 45.72)
 		)
@@
 	(wire
 		(pts
-			(xy 182.88 149.86) (xy 185.42 149.86)
+			(xy 182.88 149.86) (xy 186.69 149.86)
 		)
 		(stroke
@@
 		)
 	)
-	(hierarchical_label "TOF_R_SHUT"
+	(hierarchical_label "TOF_R_XSHUT"
 		(shape output)
 		(at 139.7 106.68 180)
@@
 		)
 	)
-	(hierarchical_label "GAUGE_INT"
-		(shape input)
-		(at 185.42 149.86 0)
-		(effects
-			(font
-				(size 1.27 1.27)
-			)
-			(justify left)
-		)
-	)
 	(hierarchical_label "ENCA_AOUT"
 		(shape input)
@@
 		)
 	)
+	(hierarchical_label "GAUGE_INT"
+		(shape input)
+		(at 186.69 127 0)
+		(effects
+			(font
+				(size 1.27 1.27)
+			)
+			(justify left)
+		)
+	)
 	(hierarchical_label "MOT_nSLEEP"
 		(shape output)
@@
 		)
 	)
+	(hierarchical_label "NEOPIXEL"
+		(shape output)
+		(at 186.69 149.86 0)
+		(effects
+			(font
+				(size 1.27 1.27)
+			)
+			(justify left)
+		)
+	)
 	(hierarchical_label "USB_DM"
 		(shape bidirectional)
@@
 		(dnp no)
 		(fields_autoplaced yes)
-		(property "Reference" "#PWR0310"
+		(property "Reference" "#PWR0311"
 			(at 242.57 93.98 0)
 			(hide yes)
@@
 			(project "projet"
 				(path "/aad9219d-d686-4d68-8dbb-b3c2b0727159/8d7235a3-ed0d-4c0c-a716-b22c65fe70a8"
-					(reference "#PWR0310")
+					(reference "#PWR0311")
 					(unit 1)
 				)
@@
 		(in_pos_files yes)
 		(dnp no)
-		(property "Reference" "#PWR0307"
+		(property "Reference" "#PWR0308"
 			(at 224.79 125.73 0)
 			(hide yes)
@@
 			(project "projet"
 				(path "/aad9219d-d686-4d68-8dbb-b3c2b0727159/8d7235a3-ed0d-4c0c-a716-b22c65fe70a8"
-					(reference "#PWR0307")
+					(reference "#PWR0308")
 					(unit 1)
 				)
@@
 		(dnp no)
 		(fields_autoplaced yes)
-		(property "Reference" "#PWR0309"
+		(property "Reference" "#PWR0310"
 			(at 242.57 71.12 0)
 			(hide yes)
@@
 			(project "projet"
 				(path "/aad9219d-d686-4d68-8dbb-b3c2b0727159/8d7235a3-ed0d-4c0c-a716-b22c65fe70a8"
-					(reference "#PWR0309")
+					(reference "#PWR0310")
 					(unit 1)
 				)
@@
 		(dnp no)
 		(fields_autoplaced yes)
-		(property "Reference" "#PWR0308"
+		(property "Reference" "#PWR0309"
 			(at 238.76 143.51 0)
 			(hide yes)
@@
 			(project "projet"
 				(path "/aad9219d-d686-4d68-8dbb-b3c2b0727159/8d7235a3-ed0d-4c0c-a716-b22c65fe70a8"
-					(reference "#PWR0308")
+					(reference "#PWR0309")
 					(unit 1)
 				)
@@
 		(dnp no)
 		(fields_autoplaced yes)
-		(property "Reference" "#PWR0311"
+		(property "Reference" "#PWR0307"
 			(at 205.74 154.94 0)
 			(hide yes)
@@
 			(project "projet"
 				(path "/aad9219d-d686-4d68-8dbb-b3c2b0727159/8d7235a3-ed0d-4c0c-a716-b22c65fe70a8"
-					(reference "#PWR0311")
+					(reference "#PWR0307")
 					(unit 1)
 				)
@@
 		(dnp no)
 		(fields_autoplaced yes)
-		(property "Reference" "R302"
+		(property "Reference" "R303"
 			(at 260.35 73.6599 0)
 			(show_name no)
@@
 			(project "projet"
 				(path "/aad9219d-d686-4d68-8dbb-b3c2b0727159/8d7235a3-ed0d-4c0c-a716-b22c65fe70a8"
-					(reference "R302")
+					(reference "R303")
 					(unit 1)
 				)
@@
 		(dnp no)
 		(fields_autoplaced yes)
-		(property "Reference" "R301"
+		(property "Reference" "R302"
 			(at 245.11 73.6599 0)
 			(show_name no)
@@
 			(project "projet"
 				(path "/aad9219d-d686-4d68-8dbb-b3c2b0727159/8d7235a3-ed0d-4c0c-a716-b22c65fe70a8"
-					(reference "R301")
+					(reference "R302")
 					(unit 1)
 				)
@@
 		(in_pos_files yes)
 		(dnp no)
-		(property "Reference" "R303"
+		(property "Reference" "R301"
 			(at 212.344 140.97 0)
 			(show_name no)
@@
 			(project "projet"
 				(path "/aad9219d-d686-4d68-8dbb-b3c2b0727159/8d7235a3-ed0d-4c0c-a716-b22c65fe70a8"
-					(reference "R303")
+					(reference "R301")
 					(unit 1)
 				)

Commit message: Correction empreintes et références JLCPCB
Parts:
- C305: footprint Capacitor_SMD:C_0402_1005Metric -> Capacitor_SMD:C_0603_1608Metric
- C308, C309: footprint Capacitor_SMD:C_0603_1608Metric -> Capacitor_SMD:C_0402_1005Metric
- J301: JLCPCB Part# (none) -> C2935955
- J302: footprint Connector_Audio:Jack_XLR_Neutrik_NC3FAAH_Horizontal -> Connector_PinHeader_2.54mm:PinHeader_1x03_P2.54mm_Vertical
