File: hardware/Projet Wall E/projet/alim.kicad_sch (KiCad schematic)
At the start: 42 parts, among them J2 USB_C_Receptacle_USB2.0_16P, J6 Conn_01x02, Q1 2SK3019, Q2 MMDT5401, Q3 DMP3099L, U1 BQ25896RTW, U2 AP2112K-3.3, U3 BQ27220YZFR, U6 USBLC6-2SC6

Commit message: Corrections alim
Parts:
- C1, C10, C11, C2, C3, C5, C7: JLCPCB Part# (none) -> C19702; JLCPCB Parts C19702 -> (none)
- C13: JLCPCB Part# (none) -> C12530; JLCPCB Parts C12530 -> (none)
- C14, C9: JLCPCB Part# (none) -> C52923; JLCPCB Parts C52923 -> (none)
- C4: JLCPCB Part# (none) -> C307434; JLCPCB Parts C307434 -> (none)
- C8: JLCPCB Part# (none) -> C19666; JLCPCB Parts C19666 -> (none)
- D1: JLCPCB Part# (none) -> C2286; JLCPCB Parts C2286 -> (none)
- D2: JLCPCB Part# (none) -> C81598; JLCPCB Parts C81598 -> (none)
- F1: JLCPCB Part# (none) -> C545216; JLCPCB Parts C545216 -> (none)
- J2: JLCPCB Part# (none) -> C165948; JLCPCB Parts C165948 -> (none)
- J6: JLCPCB Part# (none) -> C295747; JLCPCB Parts C295747 -> (none)
- L1: JLCPCB Part# (none) -> C435273; JLCPCB Parts C435273 -> (none)
- Q1: JLCPCB Part# (none) -> C261283; JLCPCB Parts C261283 -> (none)
- Q2: JLCPCB Part# (none) -> C460236; JLCPCB Parts C460236 -> (none)
- Q3: JLCPCB Part# (none) -> C155244; JLCPCB Parts C155244 -> (none)
- R1: JLCPCB Part# (none) -> C25879; JLCPCB Parts C25879 -> (none)
- R10, R9: JLCPCB Part# (none) -> C25905; JLCPCB Parts C25905 -> (none)
- R11, R13, R30, R5, R7, R8: JLCPCB Part# (none) -> C25744; JLCPCB Parts C25744 -> (none)
- R12: JLCPCB Part# (none) -> C98889; JLCPCB Parts C98889 -> (none)
- R2, R3: JLCPCB Part# (none) -> C25867; JLCPCB Parts C25867 -> (none)
- R20, R32: JLCPCB Part# (none) -> C25741; JLCPCB Parts C25741 -> (none)
- R31: JLCPCB Part# (none) -> C25076; JLCPCB Parts C25076 -> (none)
- R4: JLCPCB Part# (none) -> C25900; JLCPCB Parts C25900 -> (none)
- R6: JLCPCB Part# (none) -> C25117; JLCPCB Parts C25117 -> (none)
- U1: JLCPCB Part# (none) -> C181475; JLCPCB Parts C181475 -> (none)
- U2: JLCPCB Part# (none) -> C51118; JLCPCB Parts C51118 -> (none)
- U3: JLCPCB Part# (none) -> C528617; JLCPCB Parts C528617 -> (none)
- U6: JLCPCB Part# (none) -> C7519; JLCPCB Parts C7519 -> (none)
Changed lines of the file:
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@@
 			)
 		)
-		(property "JLCPCB Parts" "C19702"
+		(property "JLCPCB Part#" "C19702"
 			(at 238.76 59.69 0)
 			(hide yes)
@@
 			)
 		)
-		(property "JLCPCB Parts" "C25867"
+		(property "JLCPCB Part#" "C25867"
 			(at 176.53 30.48 0)
 			(hide yes)
@@
 			)
 		)
-		(property "JLCPCB Parts" "C19702"
+		(property "JLCPCB Part#" "C19702"
 			(at 227.33 88.9 0)
 			(hide yes)
@@
 			)
 		)
-		(property "JLCPCB Parts" "C261283"
+		(property "JLCPCB Part#" "C261283"
 			(at 154.94 76.2 0)
 			(hide yes)
@@
 			)
 		)
-		(property "JLCPCB Parts" "C25905"
+		(property "JLCPCB Part#" "C25905"
 			(at 93.98 48.26 0)
 			(hide yes)
@@
 			)
 		)
-		(property "JLCPCB Parts" "C25076"
+		(property "JLCPCB Part#" "C25076"
 			(at 137.16 76.2 90)
 			(hide yes)
@@
 			)
 		)
-		(property "JLCPCB Parts" "C25879"
+		(property "JLCPCB Part#" "C25879"
 			(at 214.63 35.56 0)
 			(hide yes)
@@
 			)
 		)
-		(property "JLCPCB Parts" "C98889"
+		(property "JLCPCB Part#" "C98889"
 			(at 232.41 71.12 0)
 			(hide yes)
@@
 			)
 		)
-		(property "JLCPCB Parts" "C25117"
+		(property "JLCPCB Part#" "C25117"
 			(at 187.96 81.28 0)
 			(hide yes)
@@
 			)
 		)
-		(property "JLCPCB Parts" "C460236"
+		(property "JLCPCB Part#" "C460236"
 			(at 173.99 133.35 0)
 			(hide yes)
@@
 			)
 		)
-		(property "JLCPCB Parts" "C155244"
+		(property "JLCPCB Part#" "C155244"
 			(at 158.75 118.11 90)
 			(hide yes)
@@
 			)
 		)
-		(property "JLCPCB Parts" "C19666"
+		(property "JLCPCB Part#" "C19666"
 			(at 219.71 95.25 0)
 			(hide yes)
@@
 			)
 		)
-		(property "JLCPCB Parts" "C2286"
+		(property "JLCPCB Part#" "C2286"
 			(at 214.63 24.13 90)
 			(hide yes)
@@
 			)
 		)
-		(property "JLCPCB Parts" "C19702"
+		(property "JLCPCB Part#" "C19702"
 			(at 30.48 110.49 0)
 			(hide yes)
@@
 			)
 		)
-		(property "JLCPCB Parts" "C52923"
+		(property "JLCPCB Part#" "C52923"
 			(at 158.75 45.72 0)
 			(hide yes)
@@
 			)
 		)
-		(property "JLCPCB Parts" "C25744"
+		(property "JLCPCB Part#" "C25744"
 			(at 147.32 87.63 0)
 			(hide yes)
@@
 			)
 		)
-		(property "JLCPCB Parts" "C19702"
+		(property "JLCPCB Part#" "C19702"
 			(at 234.95 88.9 0)
 			(hide yes)
@@
 			)
 		)
-		(property "JLCPCB Parts" "C25744"
+		(property "JLCPCB Part#" "C25744"
 			(at 214.63 91.44 0)
 			(hide yes)
@@
 			)
 		)
-		(property "JLCPCB Parts" "C460236"
+		(property "JLCPCB Part#" "C460236"
 			(at 156.21 133.35 0)
 			(hide yes)
@@
 			)
 		)
-		(property "JLCPCB Parts" "C25867"
+		(property "JLCPCB Part#" "C25867"
 			(at 181.61 30.48 0)
 			(hide yes)
@@
 			)
 		)
-		(property "JLCPCB Parts" "C25744"
+		(property "JLCPCB Part#" "C25744"
 			(at 214.63 81.28 0)
 			(hide yes)
@@
 			)
 		)
-		(property "JLCPCB Parts" "C25744"
+		(property "JLCPCB Part#" "C25744"
 			(at 93.98 154.94 90)
 			(hide yes)
@@
 			)
 		)
-		(property "JLCPCB Parts" "C181475"
+		(property "JLCPCB Part#" "C181475"
 			(at 201.93 58.42 0)
 			(hide yes)
@@
 			)
 		)
-		(property "JLCPCB Parts" "C12530"
+		(property "JLCPCB Part#" "C12530"
 			(at 110.49 152.4 0)
 			(hide yes)
@@
 			)
 		)
-		(property "JLCPCB Parts" "C25900"
+		(property "JLCPCB Part#" "C25900"
 			(at 170.18 30.48 0)
 			(hide yes)
@@
 			)
 		)
-		(property "JLCPCB Parts" "C25905"
+		(property "JLCPCB Part#" "C25905"
 			(at 85.09 48.26 0)
 			(hide yes)
@@
 			)
 		)
-		(property "JLCPCB Parts" "C52923"
+		(property "JLCPCB Part#" "C52923"
 			(at 35.56 149.86 0)
 			(hide yes)
@@
 			)
 		)
-		(property "JLCPCB Parts" "C7519"
+		(property "JLCPCB Part#" "C7519"
 			(at 86.36 69.85 0)
 			(hide yes)
@@
 			)
 		)
-		(property "JLCPCB Parts" "C25744"
+		(property "JLCPCB Part#" "C25744"
 			(at 143.51 63.5 0)
 			(hide yes)
@@
 			)
 		)
-		(property "JLCPCB Parts" "C545216"
+		(property "JLCPCB Part#" "C545216"
 			(at 240.03 80.01 90)
 			(hide yes)
@@
 			)
 		)
-		(property "JLCPCB Parts" "C81598"
+		(property "JLCPCB Part#" "C81598"
 			(at 139.7 128.27 90)
 			(hide yes)
@@
 			)
 		)
-		(property "JLCPCB Parts" "C307434"
+		(property "JLCPCB Part#" "C307434"
 			(at 220.98 57.15 0)
 			(hide yes)
@@
 			)
 		)
-		(property "JLCPCB Parts" "C19702"
+		(property "JLCPCB Part#" "C19702"
 			(at 58.42 109.22 0)
 			(hide yes)
@@
 			)
 		)
-		(property "JLCPCB Parts" "C25741"
+		(property "JLCPCB Part#" "C25741"
 			(at 176.53 147.32 0)
 			(hide yes)
@@
 			)
 		)
-		(property "JLCPCB Parts" "C51118"
+		(property "JLCPCB Part#" "C51118"
 			(at 45.72 105.41 0)
 			(hide yes)
@@
 			)
 		)
-		(property "JLCPCB Parts" "C295747"
+		(property "JLCPCB Part#" "C295747"
 			(at 251.46 80.01 0)
 			(hide yes)
@@
 			)
 		)
-		(property "JLCPCB Parts" "C528617"
+		(property "JLCPCB Part#" "C528617"
 			(at 67.31 154.94 0)
 			(hide yes)
@@
 			)
 		)
-		(property "JLCPCB Parts" "C435273"
+		(property "JLCPCB Part#" "C435273"
 			(at 229.87 53.34 90)
 			(hide yes)
@@
 			)
 		)
-		(property "JLCPCB Parts" "C25744"
+		(property "JLCPCB Part#" "C25744"
 			(at 48.26 173.99 0)
 			(hide yes)
@@
 			)
 		)
-		(property "JLCPCB Parts" "C25741"
+		(property "JLCPCB Part#" "C25741"
 			(at 153.67 148.59 0)
 			(hide yes)
@@
 			)
 		)
-		(property "JLCPCB Parts" "C165948"
+		(property "JLCPCB Part#" "C165948"
 			(at 49.53 50.8 0)
 			(hide yes)
@@
 			)
 		)
-		(property "JLCPCB Parts" "C19702"
+		(property "JLCPCB Part#" "C19702"
 			(at 260.35 59.69 0)
 			(hide yes)
@@
 			)
 		)
-		(property "JLCPCB Parts" "C19702"
+		(property "JLCPCB Part#" "C19702"
 			(at 248.92 59.69 0)
 			(hide yes)

Commit message: Annotation par feuille + références JLCPCB Part #
Parts:
- renumbered C10 to C201, C14 to C202, C11 to C203, C13 to C204, C9 to C205, C8 to C206, C4 to C207, C5 to C208, C1 to C209, C2 to C210, C3 to C211, C7 to C212, D2 to D201, D1 to D202, F1 to F201, J2 to J201, J6 to J202, L1 to L201, Q1 to Q201, Q2 to Q202, Q3 to Q203, R11 to R201, R9 to R202, R10 to R203, R13 to R204, R31 to R205, R30 to R206, R5 to R207, R20 to R208, R4 to R209, R3 to R210, R32 to R211, R2 to R212, R6 to R213, R1 to R214, R7 to R215, R8 to R216, R12 to R217, U2 to U201, U3 to U202, U6 to U203, U1 to U204
