File: hardware/Projet Wall E/projet/alim.kicad_sch (KiCad schematic)
At the start: 42 parts, among them J201 USB_C_Receptacle_USB2.0_16P, J202 Conn_01x02, Q201 2SK3019, Q202 MMDT5401, Q203 DMP3099L, U201 AP2112K-3.3, U202 BQ27220YZFR, U203 USBLC6-2SC6, U204 BQ25896RTW

Commit message: Modifs schématique
Parts:
- removed D201: D, Diode_SMD:D_SOD-523, symbol Device:D
- added D201: LED, LED_SMD:LED_0201_0603Metric, symbol wall_e:LED
- added R218: 2k2, Resistor_SMD:R_0402_1005Metric, symbol wall_e:R
Connections:
- net +5V_USB: now also C205.1, U204.1 (VBUS)
- net CHG_PG: now also R218.2
- net VBUS: no longer C205.1, U204.1 (VBUS)
- net VSYS: now also D201.2 (A)
- new net: D201.1 (K), R218.1

Commit message: Schéma : 0 erreur ERC, pinout MCU finalisé + config .ioc
Parts:
- renumbered R218 to R214, R214 to R215, R215 to R216, R216 to R217, R217 to R218
Changed lines of the file:
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@@
 	(wire
 		(pts
-			(xy 158.75 40.64) (xy 146.05 40.64)
-		)
-		(stroke
-			(width 0)
-			(type default)
-		)
-	)
-	(wire
-		(pts
 			(xy 158.75 50.8) (xy 158.75 49.53)
 		)
@@
 	(wire
 		(pts
-			(xy 146.05 38.1) (xy 146.05 40.64)
-		)
-		(stroke
-			(width 0)
-			(type default)
-		)
-	)
-	(wire
-		(pts
 			(xy 74.93 72.39) (xy 81.28 72.39)
 		)
@@
 		(dnp no)
 		(fields_autoplaced yes)
-		(property "Reference" "R214"
+		(property "Reference" "R215"
 			(at 217.17 34.2899 0)
 			(show_name no)
@@
 			(project "projet"
 				(path "/aad9219d-d686-4d68-8dbb-b3c2b0727159/bd811c64-dff7-4046-86a6-8e854625b7a5"
-					(reference "R214")
+					(reference "R215")
 					(unit 1)
 				)
@@
 		(in_pos_files yes)
 		(dnp no)
-		(property "Reference" "R217"
+		(property "Reference" "R218"
 			(at 235.204 67.564 0)
 			(show_name no)
@@
 			(project "projet"
 				(path "/aad9219d-d686-4d68-8dbb-b3c2b0727159/bd811c64-dff7-4046-86a6-8e854625b7a5"
-					(reference "R217")
+					(reference "R218")
 					(unit 1)
 				)
@@
 		(dnp no)
 		(fields_autoplaced yes)
-		(property "Reference" "#PWR0227"
+		(property "Reference" "#PWR0228"
 			(at 219.71 106.68 0)
 			(hide yes)
@@
 			(project "projet"
 				(path "/aad9219d-d686-4d68-8dbb-b3c2b0727159/bd811c64-dff7-4046-86a6-8e854625b7a5"
-					(reference "#PWR0227")
+					(reference "#PWR0228")
 					(unit 1)
 				)
@@
 		(in_pos_files yes)
 		(dnp no)
-		(property "Reference" "#PWR0231"
+		(property "Reference" "#PWR0232"
 			(at 260.35 71.12 0)
 			(hide yes)
@@
 			(project "projet"
 				(path "/aad9219d-d686-4d68-8dbb-b3c2b0727159/bd811c64-dff7-4046-86a6-8e854625b7a5"
-					(reference "#PWR0231")
+					(reference "#PWR0232")
 					(unit 1)
 				)
@@
 		(in_pos_files yes)
 		(dnp no)
-		(property "Reference" "R216"
+		(property "Reference" "R217"
 			(at 211.836 87.884 0)
 			(show_name no)
@@
 			(project "projet"
 				(path "/aad9219d-d686-4d68-8dbb-b3c2b0727159/bd811c64-dff7-4046-86a6-8e854625b7a5"
-					(reference "R216")
+					(reference "R217")
 					(unit 1)
 				)
@@
 		(in_pos_files yes)
 		(dnp no)
-		(property "Reference" "R215"
+		(property "Reference" "R216"
 			(at 214.122 77.978 0)
 			(show_name no)
@@
 			(project "projet"
 				(path "/aad9219d-d686-4d68-8dbb-b3c2b0727159/bd811c64-dff7-4046-86a6-8e854625b7a5"
-					(reference "R215")
+					(reference "R216")
 					(unit 1)
 				)
@@
 		(dnp no)
 		(fields_autoplaced yes)
-		(property "Reference" "#PWR0224"
+		(property "Reference" "#PWR0225"
 			(at 201.93 87.63 0)
 			(hide yes)
@@
 			(project "projet"
 				(path "/aad9219d-d686-4d68-8dbb-b3c2b0727159/bd811c64-dff7-4046-86a6-8e854625b7a5"
-					(reference "#PWR0224")
+					(reference "#PWR0225")
 					(unit 1)
 				)
@@
 		(dnp no)
 		(fields_autoplaced yes)
-		(property "Reference" "#PWR0226"
+		(property "Reference" "#PWR0227"
 			(at 214.63 106.68 0)
 			(hide yes)
@@
 			(project "projet"
 				(path "/aad9219d-d686-4d68-8dbb-b3c2b0727159/bd811c64-dff7-4046-86a6-8e854625b7a5"
-					(reference "#PWR0226")
+					(reference "#PWR0227")
 					(unit 1)
 				)
@@
 	)
 	(symbol
-		(lib_id "power:PWR_FLAG")
-		(at 146.05 38.1 0)
-		(unit 1)
-		(body_style 1)
-		(exclude_from_sim no)
-		(in_bom yes)
-		(on_board yes)
-		(in_pos_files yes)
-		(dnp no)
-		(fields_autoplaced yes)
-		(property "Reference" "#FLG0203"
-			(at 146.05 36.195 0)
-			(hide yes)
-			(show_name no)
-			(do_not_autoplace no)
-			(effects
-				(font
-					(size 1.27 1.27)
-				)
-			)
-		)
-		(property "Value" "PWR_FLAG"
-			(at 146.05 33.02 0)
-			(show_name no)
-			(do_not_autoplace no)
-			(effects
-				(font
-					(size 1.27 1.27)
-				)
-			)
-		)
-		(property "Footprint" ""
-			(at 146.05 38.1 0)
-			(hide yes)
-			(show_name no)
-			(do_not_autoplace no)
-			(effects
-				(font
-					(size 1.27 1.27)
-				)
-			)
-		)
-		(property "Datasheet" ""
-			(at 146.05 38.1 0)
-			(hide yes)
-			(show_name no)
-			(do_not_autoplace no)
-			(effects
-				(font
-					(size 1.27 1.27)
-				)
-			)
-		)
-		(property "Description" "Special symbol for telling ERC where power comes from"
-			(at 146.05 38.1 0)
-			(hide yes)
-			(show_name no)
-			(do_not_autoplace no)
-			(effects
-				(font
-					(size 1.27 1.27)
-				)
-			)
-		)
-		(pin "1"
-		)
-		(instances
-			(project "projet"
-				(path "/aad9219d-d686-4d68-8dbb-b3c2b0727159/bd811c64-dff7-4046-86a6-8e854625b7a5"
-					(reference "#FLG0203")
-					(unit 1)
-				)
-			)
-		)
-	)
-	(symbol
 		(lib_id "power:+5V")
 		(at 86.36 62.23 0)
@@
 		(in_pos_files yes)
 		(dnp no)
-		(property "Reference" "#PWR0229"
+		(property "Reference" "#PWR0230"
 			(at 243.84 48.26 0)
 			(hide yes)
@@
 			(project "projet"
 				(path "/aad9219d-d686-4d68-8dbb-b3c2b0727159/bd811c64-dff7-4046-86a6-8e854625b7a5"
-					(reference "#PWR0229")
+					(reference "#PWR0230")
 					(unit 1)
 				)
@@
 		(dnp no)
 		(fields_autoplaced yes)
-		(property "Reference" "R218"
+		(property "Reference" "R214"
 			(at 193.04 30.4799 0)
 			(show_name no)
@@
 			(project "projet"
 				(path "/aad9219d-d686-4d68-8dbb-b3c2b0727159/bd811c64-dff7-4046-86a6-8e854625b7a5"
-					(reference "R218")
+					(reference "R214")
 					(unit 1)
 				)
@@
 		(in_pos_files yes)
 		(dnp no)
-		(property "Reference" "#PWR0225"
+		(property "Reference" "#PWR0226"
 			(at 214.63 21.59 0)
 			(hide yes)
@@
 			(project "projet"
 				(path "/aad9219d-d686-4d68-8dbb-b3c2b0727159/bd811c64-dff7-4046-86a6-8e854625b7a5"
-					(reference "#PWR0225")
+					(reference "#PWR0226")
 					(unit 1)
 				)
@@
 		(in_pos_files yes)
 		(dnp no)
-		(property "Reference" "#PWR0230"
+		(property "Reference" "#PWR0231"
 			(at 243.84 72.39 0)
 			(hide yes)
@@
 			(project "projet"
 				(path "/aad9219d-d686-4d68-8dbb-b3c2b0727159/bd811c64-dff7-4046-86a6-8e854625b7a5"
-					(reference "#PWR0230")
+					(reference "#PWR0231")
 					(unit 1)
 				)
@@
 		(in_pos_files yes)
 		(dnp no)
-		(property "Reference" "#PWR0232"
+		(property "Reference" "#PWR0224"
 			(at 190.5 21.59 0)
 			(hide yes)
@@
 			(project "projet"
 				(path "/aad9219d-d686-4d68-8dbb-b3c2b0727159/bd811c64-dff7-4046-86a6-8e854625b7a5"
-					(reference "#PWR0232")
+					(reference "#PWR0224")
 					(unit 1)
 				)
@@
 		(dnp no)
 		(fields_autoplaced yes)
-		(property "Reference" "#PWR0228"
+		(property "Reference" "#PWR0229"
 			(at 234.95 101.6 0)
 			(hide yes)
@@
 			(project "projet"
 				(path "/aad9219d-d686-4d68-8dbb-b3c2b0727159/bd811c64-dff7-4046-86a6-8e854625b7a5"
-					(reference "#PWR0228")
+					(reference "#PWR0229")
 					(unit 1)
 				)

Commit message: Correction empreintes et références JLCPCB
Parts:
- D201, D202: footprint LED_SMD:LED_0201_0603Metric -> LED_SMD:LED_0603_1608Metric
- L201: JLCPCB Part# C435273 -> C316359
- R209, R210, R212: footprint Resistor_SMD:R_01005_0402Metric -> Resistor_SMD:R_0402_1005Metric

Commit message: verification finale effectue
Parts:
- C202: value 1µ -> 1u
Changed lines of the file:
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@@
 			)
 		)
-		(property "Value" "1µ"
+		(property "Value" "1u"
 			(at 31.496 152.4 0)
 			(show_name no)

Commit message: Ajout points de test + plans de masse PCB
Parts:
- added TP201, TP210, TP211: GND, TestPoint:TestPoint_Pad_D1.5mm, symbol Connector:TestPoint
- added TP202: VSYS, TestPoint:TestPoint_Pad_D1.0mm, symbol Connector:TestPoint
- added TP203: +3.3V, TestPoint:TestPoint_Pad_D1.0mm, symbol Connector:TestPoint
- added TP204: +5V_USB, TestPoint:TestPoint_Pad_D1.0mm, symbol Connector:TestPoint
- added TP205: VBUS, TestPoint:TestPoint_Pad_D1.0mm, symbol Connector:TestPoint
- added TP206: BAT, TestPoint:TestPoint_Pad_D1.0mm, symbol Connector:TestPoint
- added TP207: SCL, TestPoint:TestPoint_Pad_D1.0mm, symbol Connector:TestPoint
- added TP208: SDA, TestPoint:TestPoint_Pad_D1.0mm, symbol Connector:TestPoint
- added TP209: CHG_INT, TestPoint:TestPoint_Pad_D1.0mm, symbol Connector:TestPoint
Connections:
- net +3.3V: now also TP203.1
- net +5V_USB: now also TP204.1
- net BAT: now also TP206.1
- net CHG_INT: now also TP209.1
- net GND: now also TP201.1, TP210.1, TP211.1
- net SCL: now also TP207.1
- net SDA: now also TP208.1
- net VBUS: now also TP205.1
- net VSYS: now also TP202.1

Commit message: PCB : placement composants et points de test
Connections:
- net at C206.2, U204.22 (REGN): now also R216.2; no longer R216.1, R217.1
- net at U204.11 (TS): now also R216.1, R217.1; no longer R216.2
Other:
- moved on the sheet: R216, R217
Changed lines of the file:
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@@
 	)
 	(junction
+		(at 217.17 71.12)
+		(diameter 0)
+		(color 0 0 0 0)
+	)
+	(junction
 		(at 68.58 54.61)
 		(diameter 0)
@@
 	)
 	(junction
-		(at 219.71 86.36)
+		(at 214.63 86.36)
 		(diameter 0)
 		(color 0 0 0 0)
@@
 	)
 	(junction
-		(at 214.63 86.36)
-		(diameter 0)
-		(color 0 0 0 0)
-	)
-	(junction
 		(at 45.72 115.57)
 		(diameter 0)
@@
 	(wire
 		(pts
+			(xy 217.17 71.12) (xy 217.17 73.66)
+		)
+		(stroke
+			(width 0)
+			(type default)
+		)
+	)
+	(wire
+		(pts
 			(xy 214.63 27.94) (xy 214.63 31.75)
 		)
@@
 	(wire
 		(pts
+			(xy 214.63 86.36) (xy 214.63 90.17)
+		)
+		(stroke
+			(width 0)
+			(type default)
+		)
+	)
+	(wire
+		(pts
 			(xy 139.7 115.57) (xy 153.67 115.57)
 		)
@@
 	(wire
 		(pts
-			(xy 219.71 71.12) (xy 212.09 71.12)
+			(xy 212.09 71.12) (xy 217.17 71.12)
 		)
 		(stroke
@@
 	(wire
 		(pts
-			(xy 212.09 76.2) (xy 214.63 76.2)
-		)
-		(stroke
-			(width 0)
-			(type default)
-		)
-	)
-	(wire
-		(pts
 			(xy 156.21 91.44) (xy 156.21 92.71)
 		)
@@
 	(wire
 		(pts
-			(xy 214.63 85.09) (xy 214.63 86.36)
+			(xy 217.17 81.28) (xy 217.17 86.36)
 		)
 		(stroke
@@
 	(wire
 		(pts
-			(xy 219.71 86.36) (xy 214.63 86.36)
+			(xy 82.55 154.94) (xy 88.9 154.94)
 		)
 		(stroke
@@
 	(wire
 		(pts
-			(xy 82.55 154.94) (xy 88.9 154.94)
+			(xy 212.09 76.2) (xy 212.09 86.36)
 		)
 		(stroke
@@
 	(wire
 		(pts
-			(xy 214.63 86.36) (xy 214.63 87.63)
+			(xy 147.32 91.44) (xy 156.21 91.44)
 		)
 		(stroke
@@
 	(wire
 		(pts
-			(xy 147.32 91.44) (xy 156.21 91.44)
+			(xy 48.26 179.07) (xy 48.26 177.8)
 		)
 		(stroke
@@
 	(wire
 		(pts
-			(xy 48.26 179.07) (xy 48.26 177.8)
+			(xy 68.58 55.88) (xy 64.77 55.88)
 		)
 		(stroke
@@
 	(wire
 		(pts
-			(xy 68.58 55.88) (xy 64.77 55.88)
+			(xy 157.48 68.58) (xy 170.18 68.58)
 		)
 		(stroke
@@
 	(wire
 		(pts
-			(xy 157.48 68.58) (xy 170.18 68.58)
+			(xy 153.67 152.4) (xy 153.67 156.21)
 		)
 		(stroke
@@
 	(wire
 		(pts
-			(xy 153.67 152.4) (xy 153.67 156.21)
+			(xy 217.17 71.12) (xy 219.71 71.12)
 		)
 		(stroke
@@
 	(wire
 		(pts
+			(xy 217.17 86.36) (xy 214.63 86.36)
+		)
+		(stroke
+			(width 0)
+			(type default)
+		)
+	)
+	(wire
+		(pts
 			(xy 191.77 76.2) (xy 187.96 76.2)
 		)
@@
 	(wire
 		(pts
+			(xy 212.09 86.36) (xy 214.63 86.36)
+		)
+		(stroke
+			(width 0)
+			(type default)
+		)
+	)
+	(wire
+		(pts
 			(xy 153.67 128.27) (xy 151.13 128.27)
 		)
@@
 	(wire
 		(pts
-			(xy 214.63 95.25) (xy 214.63 100.33)
+			(xy 214.63 97.79) (xy 214.63 100.33)
 		)
 		(stroke
@@
 	(wire
 		(pts
-			(xy 219.71 71.12) (xy 219.71 86.36)
+			(xy 219.71 71.12) (xy 219.71 91.44)
 		)
 		(stroke
@@
 	(wire
 		(pts
-			(xy 214.63 76.2) (xy 214.63 77.47)
-		)
-		(stroke
-			(width 0)
-			(type default)
-		)
-	)
-	(wire
-		(pts
 			(xy 30.48 102.87) (xy 30.48 105.41)
 		)
@@
 	(wire
 		(pts
-			(xy 219.71 86.36) (xy 219.71 91.44)
-		)
-		(stroke
-			(width 0)
-			(type default)
-		)
-	)
-	(wire
-		(pts
 			(xy 163.83 115.57) (xy 176.53 115.57)
 		)
@@
 	(symbol
 		(lib_id "wall_e:R")
-		(at 214.63 91.44 0)
+		(at 214.63 93.98 0)
 		(unit 1)
 		(body_style 1)
@@
 		(dnp no)
 		(property "Reference" "R217"
-			(at 211.836 87.884 0)
+			(at 211.836 90.424 0)
 			(show_name no)
 			(do_not_autoplace no)
@@
 		)
 		(property "Value" "10k"
-			(at 210.566 95.25 0)
+			(at 210.566 97.79 0)
 			(show_name no)
 			(do_not_autoplace no)
@@
 		)
 		(property "Footprint" "Resistor_SMD:R_0402_1005Metric"
-			(at 212.852 91.44 90)
+			(at 212.852 93.98 90)
 			(hide yes)
 			(show_name no)
@@
 		)
 		(property "Datasheet" ""
-			(at 214.63 91.44 0)
+			(at 214.63 93.98 0)
 			(hide yes)
 			(show_name no)
@@
 		)
 		(property "Description" "Resistor"
-			(at 214.63 91.44 0)
+			(at 214.63 93.98 0)
 			(hide yes)
 			(show_name no)
@@
 		)
 		(property "JLCPCB Part#" "C25744"
-			(at 214.63 91.44 0)
+			(at 214.63 93.98 0)
 			(hide yes)
 			(show_name no)
@@
 		)
 		(property "KLC_S3.3" ""
-			(at 214.63 91.44 0)
+			(at 214.63 93.98 0)
 			(hide yes)
 			(show_name no)
@@
 		)
 		(property "KLC_S4.1" ""
-			(at 214.63 91.44 0)
+			(at 214.63 93.98 0)
 			(hide yes)
 			(show_name no)
@@
 		)
 		(property "Sim.Device" ""
-			(at 214.63 91.44 0)
+			(at 214.63 93.98 0)
 			(hide yes)
 			(show_name no)
@@
 	(symbol
 		(lib_id "wall_e:R")
-		(at 214.63 81.28 180)
+		(at 217.17 77.47 180)
 		(unit 1)
 		(body_style 1)
@@
 		(dnp no)
 		(property "Reference" "R216"
-			(at 214.122 77.978 0)
+			(at 216.662 74.168 0)
 			(show_name no)
 			(do_not_autoplace no)
@@
 		)
 		(property "Value" "10k"
-			(at 213.868 84.836 0)
+			(at 216.408 81.026 0)
 			(show_name no)
 			(do_not_autoplace no)
@@
 		)
 		(property "Footprint" "Resistor_SMD:R_0402_1005Metric"
-			(at 216.408 81.28 90)
+			(at 218.948 77.47 90)
 			(hide yes)
 			(show_name no)
@@
 		)
 		(property "Datasheet" ""
-			(at 214.63 81.28 0)
+			(at 217.17 77.47 0)
 			(hide yes)
 			(show_name no)
@@
 		)
 		(property "Description" "Resistor"
-			(at 214.63 81.28 0)
+			(at 217.17 77.47 0)
 			(hide yes)
 			(show_name no)
@@
 		)
 		(property "JLCPCB Part#" "C25744"
-			(at 214.63 81.28 0)
+			(at 217.17 77.47 0)
 			(hide yes)
 			(show_name no)
@@
 		)
 		(property "KLC_S3.3" ""
-			(at 214.63 81.28 0)
+			(at 217.17 77.47 0)
 			(hide yes)
 			(show_name no)
@@
 		)
 		(property "KLC_S4.1" ""
-			(at 214.63 81.28 0)
+			(at 217.17 77.47 0)
 			(hide yes)
 			(show_name no)
@@
 		)
 		(property "Sim.Device" ""
-			(at 214.63 81.28 0)
+			(at 217.17 77.47 0)
 			(hide yes)
 			(show_name no)

Commit message: correction erreur drc
Changed lines of the file:
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@@
 	)
 	(junction
+		(at 68.58 35.56)
+		(diameter 0)
+		(color 0 0 0 0)
+	)
+	(junction
 		(at 180.34 87.63)
 		(diameter 0)
@@
 	(wire
 		(pts
+			(xy 78.74 30.48) (xy 78.74 35.56)
+		)
+		(stroke
+			(width 0)
+			(type default)
+		)
+	)
+	(wire
+		(pts
 			(xy 214.63 27.94) (xy 214.63 31.75)
 		)
@@
 	(wire
 		(pts
+			(xy 78.74 35.56) (xy 68.58 35.56)
+		)
+		(stroke
+			(width 0)
+			(type default)
+		)
+	)
+	(wire
+		(pts
 			(xy 212.09 63.5) (xy 234.95 63.5)
 		)
@@
 					(unit 1)
 				)
+			)
+		)
+	)
+	(symbol
+		(lib_id "power:PWR_FLAG")
+		(at 78.74 30.48 0)
+		(unit 1)
+		(body_style 1)
+		(exclude_from_sim no)
+		(in_bom yes)
+		(on_board yes)
+		(in_pos_files yes)
+		(dnp no)
+		(property "Reference" "#FLG0203"
+			(at 78.74 28.575 0)
+			(hide yes)
+			(show_name no)
+			(do_not_autoplace no)
+			(effects
+				(font
+					(size 1.27 1.27)
+				)
+			)
+		)
+		(property "Value" "PWR_FLAG"
+			(at 78.74 26.416 0)
+			(show_name no)
+			(do_not_autoplace no)
+			(effects
+				(font
+					(size 1.27 1.27)
+				)
+			)
+		)
+		(property "Footprint" ""
+			(at 78.74 30.48 0)
+			(hide yes)
+			(show_name no)
+			(do_not_autoplace no)
+			(effects
+				(font
+					(size 1.27 1.27)
+				)
+			)
+		)
+		(property "Datasheet" ""
+			(at 78.74 30.48 0)
+			(hide yes)
+			(show_name no)
+			(do_not_autoplace no)
+			(effects
+				(font
+					(size 1.27 1.27)
+				)
+			)
+		)
+		(property "Description" "Special symbol for telling ERC where power comes from"
+			(at 78.74 30.48 0)
+			(hide yes)
+			(show_name no)
+			(do_not_autoplace no)
+			(effects
+				(font
+					(size 1.27 1.27)
+				)
+			)
+		)
+		(pin "1"
+		)
+		(instances
+			(project "projet"
+				(path "/aad9219d-d686-4d68-8dbb-b3c2b0727159/bd811c64-dff7-4046-86a6-8e854625b7a5"
+					(reference "#FLG0203")
+					(unit 1)
+				)

Commit message: (feat : Placement PCB 10*6cm et mise à jour TestPoint)
Parts:
- TP201: footprint TestPoint:TestPoint_Pad_D1.5mm -> TestPoint:TestPoint_Pad_D1.0mm
- TP207, TP208, TP209: footprint TestPoint:TestPoint_Pad_D1.0mm -> TestPoint:TestPoint_Loop_D2.50mm_Drill1.0mm
Changed lines of the file:
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@@
 			)
 		)
-		(property "Footprint" "TestPoint:TestPoint_Pad_D1.5mm"
+		(property "Footprint" "TestPoint:TestPoint_Pad_D1.0mm"
 			(at 260.35 160.02 0)
 			(hide yes)
@@
 			)
 		)
-		(property "Footprint" "TestPoint:TestPoint_Pad_D1.0mm"
+		(property "Footprint" "TestPoint:TestPoint_Loop_D2.50mm_Drill1.0mm"
 			(at 229.87 151.13 0)
 			(hide yes)
@@
 			)
 		)
-		(property "Footprint" "TestPoint:TestPoint_Pad_D1.0mm"
+		(property "Footprint" "TestPoint:TestPoint_Loop_D2.50mm_Drill1.0mm"
 			(at 229.87 143.51 0)
 			(hide yes)
@@
 			)
 		)
-		(property "Footprint" "TestPoint:TestPoint_Pad_D1.0mm"
+		(property "Footprint" "TestPoint:TestPoint_Loop_D2.50mm_Drill1.0mm"
 			(at 229.87 158.75 0)
 			(hide yes)
