File: hardware/Projet Wall E/projet/moteur.kicad_sch (KiCad schematic)
At the start: 11 parts, among them J401 Conn_01x06, J402 Conn_01x06, U401 DRV8833PWP

Commit message: Fichiers de fabrication : Gerbers, perçage, CPL et BOM
Parts:
- J401, J402, TP401: now left out of the parts list
Changed lines of the file:
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@@
 		(body_style 1)
 		(exclude_from_sim no)
-		(in_bom yes)
+		(in_bom no)
 		(on_board yes)
 		(in_pos_files yes)
@@
 		(body_style 1)
 		(exclude_from_sim no)
-		(in_bom yes)
+		(in_bom no)
 		(on_board yes)
 		(in_pos_files yes)
@@
 		(body_style 1)
 		(exclude_from_sim no)
-		(in_bom yes)
+		(in_bom no)
 		(on_board yes)
 		(in_pos_files yes)

Commit message: Fabrication : BOM mise à jour, CPL corrigé (rotations JLCPCB), nouvelles références Q201/Q202/R218
Parts:
- C402: value 2.2uF -> 2u2
Changed lines of the file:
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@@
 			)
 		)
-		(property "Value" "2.2uF"
+		(property "Value" "2u2"
 			(at 87.63 63.4999 0)
 			(show_name no)
