File: hardware/Projet Wall E/projet/projet.kicad_pcb (KiCad board)
At the start: 4 copper layers, 100 x 40 mm, 108 parts, among them J201 USB_C_Receptacle_USB2.0_16P, J301 Conn_ST_STDC14, Q201 2SK3019, Q202 MMDT5401, Q203 DMP3099L, U201 AP2112K-3.3, U202 BQ27220YZFR, U203 USBLC6-2SC6, U204 BQ25896RTW, U301 STM32G431RBTx, U401 DRV8833PWP, U501 SN74AHCT1G125DBVR, Y301 16MHz

Commit message: Fabrication : BOM mise à jour, CPL corrigé (rotations JLCPCB), nouvelles références Q201/Q202/R218
Parts:
- renumbered ALIM to J202
Other:
- board text added: "ALIM"
Changed lines of the file:
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@@
 		(descr "JST PH series connector, S2B-PH-SM4-TB (http://www.jst-mfg.com/product/pdf/eng/ePH.pdf)")
 		(tags "connector JST PH horizontal")
-		(property "Reference" "ALIM"
+		(property "Reference" "J202"
 			(at 0 -5.8 90)
 			(layer "F.SilkS")
@@
 			)
 		)
-		(attr smd exclude_from_pos_files)
+		(attr smd)
 		(duplicate_pad_numbers_are_jumpers no)
 		(fp_line
@@
 			)
 		)
-		(attr smd)
+		(attr smd exclude_from_pos_files)
 		(duplicate_pad_numbers_are_jumpers no)
 		(fp_line
@@
 		(layer "Edge.Cuts")
 	)
+	(gr_text "ALIM"
+		(at 114.55 85.15 90)
+		(layer "F.SilkS")
+		(effects
+			(font
+				(size 0.8 0.6)
+				(thickness 0.15)
+				(bold yes)
+			)
+			(justify left bottom)
+		)
+	)
 	(gr_text "PROJET WALL-E\nENSEA ESE 2026-2027\nTURGUT Iprahim · SDIRI Lamyae\nBEAUSON William · CHEIKH Abdellahi\nTSAMO Florette"
